File: KiCad/Hardware.kicad_sch (KiCad schematic)
At the start: 1 part

Commit message: Ver X1.0
Copied latest changes from backup project
Parts:
- added H201: Lipstick Tube, symbol Graphic:Logo_Open_Hardware_Small
- added H202: PCB, symbol Graphic:Logo_Open_Hardware_Small
- added H204: Amidon Toroid, symbol Graphic:Logo_Open_Hardware_Small
- added H205: Amidon Ferrite Bead, symbol Graphic:Logo_Open_Hardware_Small
- added H206: Cable Ties, symbol Graphic:Logo_Open_Hardware_Small
- N201: footprint (none) -> ~; Link (none) -> https://www.polycase.com/sl-42p#SL-42PMBR; Manufacturer (none) -> PolyCase; Manufacturer PN (none) -> SL-42PMBR

Commit message: Ver 1.0
Redesign of LED tuning indicator. All gerbers updated.
Parts:
- renumbered H202 to H201, H201 to H202, H204 to H203, H205 to H204, H206 to H205
Changed lines of the file:
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@@
 	(title_block
 		(title "80m Bottom-Loaded Vertical Fox Antenna")
-		(date "2026-01-02")
-		(rev "X1.0")
+		(date "2026-01-09")
+		(rev "1.0")
 	)
 	(symbol
@@
 			)
 		)
+		(property "Sim.Enable" ""
+			(at 101.6 59.69 0)
+			(effects
+				(font
+					(size 1.27 1.27)
+				)
+				(hide yes)
+			)
+		)
 		(instances
 			(project "SignalStreamer"
@@
 		(dnp no)
 		(fields_autoplaced yes)
-		(property "Reference" "H206"
+		(property "Reference" "H205"
 			(at 173.99 55.245 0)
 			(effects
@@
 				(font
 					(size 2.9972 2.9972)
+				)
+				(hide yes)
+			)
+		)
+		(property "Sim.Enable" ""
+			(at 173.99 62.23 0)
+			(effects
+				(font
+					(size 1.27 1.27)
 				)
 				(hide yes)
@@
 			(project "SignalStreamer"
 				(path "/bb5a72dd-4ae0-443a-a555-e26e42998b39/c9b73006-4888-422c-a9e5-798bf192af53"
-					(reference "H206")
+					(reference "H205")
 					(unit 1)
 				)
@@
 		(dnp no)
 		(fields_autoplaced yes)
-		(property "Reference" "H205"
+		(property "Reference" "H204"
 			(at 154.94 55.245 0)
 			(effects
@@
 				(font
 					(size 2.9972 2.9972)
+				)
+				(hide yes)
+			)
+		)
+		(property "Sim.Enable" ""
+			(at 154.94 62.23 0)
+			(effects
+				(font
+					(size 1.27 1.27)
 				)
 				(hide yes)
@@
 			(project "SignalStreamer"
 				(path "/bb5a72dd-4ae0-443a-a555-e26e42998b39/c9b73006-4888-422c-a9e5-798bf192af53"
-					(reference "H205")
+					(reference "H204")
 					(unit 1)
 				)
@@
 		(dnp no)
 		(fields_autoplaced yes)
-		(property "Reference" "H204"
+		(property "Reference" "H203"
 			(at 130.81 55.245 0)
 			(effects
@@
 				(font
 					(size 2.9972 2.9972)
+				)
+				(hide yes)
+			)
+		)
+		(property "Sim.Enable" ""
+			(at 130.81 62.23 0)
+			(effects
+				(font
+					(size 1.27 1.27)
 				)
 				(hide yes)
@@
 			(project "SignalStreamer"
 				(path "/bb5a72dd-4ae0-443a-a555-e26e42998b39/c9b73006-4888-422c-a9e5-798bf192af53"
-					(reference "H204")
+					(reference "H203")
 					(unit 1)
 				)
@@
 		(dnp no)
 		(fields_autoplaced yes)
-		(property "Reference" "H201"
+		(property "Reference" "H202"
 			(at 128.27 75.565 0)
 			(effects
@@
 				(font
 					(size 2.9972 2.9972)
+				)
+				(hide yes)
+			)
+		)
+		(property "Sim.Enable" ""
+			(at 128.27 82.55 0)
+			(effects
+				(font
+					(size 1.27 1.27)
 				)
 				(hide yes)
@@
 			(project "SignalStreamer"
 				(path "/bb5a72dd-4ae0-443a-a555-e26e42998b39/c9b73006-4888-422c-a9e5-798bf192af53"
-					(reference "H201")
+					(reference "H202")
 					(unit 1)
 				)
@@
 		(dnp no)
 		(fields_autoplaced yes)
-		(property "Reference" "#SYM203"
+		(property "Reference" "#SYM201"
 			(at 156.21 76.835 0)
 			(effects
@@
 			(project "SignalStreamer"
 				(path "/bb5a72dd-4ae0-443a-a555-e26e42998b39/c9b73006-4888-422c-a9e5-798bf192af53"
-					(reference "#SYM203")
+					(reference "#SYM201")
 					(unit 1)
 				)
@@
 		(dnp no)
 		(fields_autoplaced yes)
-		(property "Reference" "H202"
+		(property "Reference" "H201"
 			(at 101.6 76.835 0)
 			(effects
@@
 				(font
 					(size 2.9972 2.9972)
+				)
+				(hide yes)
+			)
+		)
+		(property "Sim.Enable" ""
+			(at 101.6 83.82 0)
+			(effects
+				(font
+					(size 1.27 1.27)
 				)
 				(hide yes)
@@
 			(project "SignalStreamer"
 				(path "/bb5a72dd-4ae0-443a-a555-e26e42998b39/c9b73006-4888-422c-a9e5-798bf192af53"
-					(reference "H202")
+					(reference "H201")
 					(unit 1)
 				)
