File: KiCad/Hardware.kicad_sch (KiCad schematic)
At the start: 6 parts

Commit message: Updates
Added bypass capacitors across diodes
10k pot, now wired as potentiometer
Other:
- title: 80m Bottom-Loaded Vertical Fox Antenna -> 80m Base-Loaded Vertical Fox Antenna
Changed lines of the file:
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@@
 	(paper "A4")
 	(title_block
-		(title "80m Bottom-Loaded Vertical Fox Antenna")
-		(date "2026-01-09")
-		(rev "1.0")
+		(title "80m Base-Loaded Vertical Fox Antenna")
+		(date "2026-09-28")
+		(rev "1.1")
 	)
 	(symbol

Commit message: Design Updates
Changes to improve LED illumination for better tuning indication. This will become SignalStreamer Ver 1.1. The PCB design has not yet been updated.
Parts:
- N201: footprint ~ -> (none)
Changed lines of the file:
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@@
 	(title_block
 		(title "80m Base-Loaded Vertical Fox Antenna")
-		(date "2026-09-28")
+		(date "2026-10-16")
 		(rev "1.1")
 	)
@@
 			)
 		)
-		(property "Footprint" "~"
+		(property "Footprint" ""
 			(at 102.87 58.42 0)
 			(effects
